File: SOA_examples/v/drawing.kicad_pcb (KiCad board)
At the start: 2 copper layers, 47.9 x 47.9 mm, 10 parts

Commit message: finished pcb
Parts:
- added REF**: PinHeader_2x03_P2.54mm_Vertical, Connector_PinHeader_2.54mm:PinHeader_2x03_P2.54mm_Vertical, F.Cu at (56.4, 50.0)
- moved REF** 1.30 mm to (77.5, 75.9), turned to 135 degrees
- moved REF** 1.29 mm to (61.2, 82.8), turned to 90 degrees
- moved REF** 1.27 mm to (38.4, 59.9), turned to 180 degrees
- moved REF** 1.27 mm to (83.8, 59.7), turned to 180 degrees
- moved REF** 1.08 mm to (61.0, 37.3), turned to 90 degrees
- moved REF** 1.05 mm to (77.0, 43.7), turned to 45 degrees
- moved REF** 0.76 mm to (45.0, 43.9), turned to 135 degrees
- moved REF** 0.72 mm to (45.2, 75.7), turned to 45 degrees
Routing:
- net (no net): track 161.0 -> 176.9 mm
